File: hardware/ieiunium-claritsa.sch (KiCad schematic (older format))
At the start: 31 parts

Commit message: Create netlist. Leave switch and L1 without pcb footprints. Await delivery...
Parts:
- removed XL?: CONN_3, symbol CONN_3
- added C9: 0.1u, Capacitors:CAP_0603, symbol C
- added F1: Fuse0R, Resistors:RES_0603_FUSE, symbol Fuse0R
- added TP1: SCL, PCB:TESTPOINT_1MM, symbol TESTPOINT
- added TP2: SDA, PCB:TESTPOINT_1MM, symbol TESTPOINT
- added XL1: CONN_2, Connectors:PLS-2, symbol CONN_2
- C1, C5, C6, C7, C8: renamed from C?; footprint CAP_0603 -> Capacitors:CAP_0603
- C2: renamed from C?; footprint CAP_0805 -> Capacitors:CAP_0805
- C3, C4: renamed from C?; value C -> 0.1u; footprint CAP_0603 -> Capacitors:CAP_0603
- D1: renamed from D?; footprint (none) -> LEDs:LED_0603
- D2: renamed from D?; footprint SOD-123 -> Diodes:SOD323
- DA1: renamed from DA?; footprint (none) -> SOT:SOT23-5
- DD1, DD2: renamed from DD?; footprint (none) -> LQFP_TQFP:LQFP48
- L1: renamed from L?; footprint IND_0402 -> (none)
- R1, R2, R3, R4, R5: renamed from R?; footprint RES_0603 -> Resistors:RES_0603
- TP3: renamed from TP?; value TESTPOINT -> NRST; footprint (none) -> PCB:TESTPOINT_1MM
- TP4: renamed from TP?; value TESTPOINT -> SCK; footprint (none) -> PCB:TESTPOINT_1MM
- TP5: renamed from TP?; value TESTPOINT -> SDI; footprint (none) -> PCB:TESTPOINT_1MM
- TP6: renamed from TP?; value TESTPOINT -> SDO; footprint (none) -> PCB:TESTPOINT_1MM
- TP7: renamed from TP?; value TESTPOINT -> CS; footprint (none) -> PCB:TESTPOINT_1MM
- TP8: renamed from TP?; value TESTPOINT -> INT1; footprint (none) -> PCB:TESTPOINT_1MM
- TP9: renamed from TP?; value TESTPOINT -> INT2; footprint (none) -> PCB:TESTPOINT_1MM
- XL2: renamed from XL?; footprint (none) -> Connectors:PLS-4
- XL3: renamed from XL?; footprint (none) -> Connectors:PLS-2
- XL4: renamed from XL?; footprint (none) -> Connectors:PLS-5
- gave numbers to parts that had none: 1
Connections:
- net +3.3V: now also C9.1, F1.2; no longer XL4.1
- net GND: now also C9.2, XL1.1 (P1)
- net LIS_CS: now also DD1.14 (ADC4/T14C1/DAC1/CK2/PA4); no longer DD1.29 (MCO/T1C1/CK1/PA8)
- net LIS_INT1: now also DD1.18 (PB0/T3C3/T1C2N/ADC8); no longer DD1.19 (PB1/T3C4/T1C3N/T14C1/ADC9)
- net LIS_INT2: now also DD1.19 (PB1/T3C4/T1C3N/T14C1/ADC9); no longer DD1.20 (PB2)
- net at R1.1: now also DD1.40 (PB4/T3C1/MISO1); no longer DD1.18 (PB0/T3C3/T1C2N/ADC8)
- net DBG_TX: now reaches DD1.30 (T1C2/TX1/PA9)
- net DBG_TX: now also XL1.2 (PM)
- net at DD1.45 (PB8/SCL1/T16C1): now also TP1.1
- net at DD1.46 (PB9/SDA1/T17C1/IR_OUT): now also TP2.1
- new net: F1.1, XL4.1
- no-connect marks 25 -> 24
Other:
- moved on the sheet: D1, DD2, R1, TP3, TP4, TP5, TP6, TP7, TP8, TP9

Commit message: + PCB with footprints
Parts:
- C1: footprint Capacitors:CAP_0603 -> Capacitors:CAP_0805
- DD2: footprint LQFP_TQFP:LQFP48 -> LGA:16_3X3
- L1: footprint (none) -> Inductors:CD_type_6.0X5.5
- SW1: footprint (none) -> Socket_Strips:Socket_Strip_Straight_1x03_Pitch2.54mm
- XL1: footprint Connectors:PLS-2 -> Socket_Strips:Socket_Strip_Straight_1x02_Pitch2.54mm
- XL2: footprint Connectors:PLS-4 -> Socket_Strips:Socket_Strip_Straight_1x04_Pitch2.54mm
- XL3: footprint Connectors:PLS-2 -> Installation:BH-6_CR2032
- XL4: footprint Connectors:PLS-5 -> Socket_Strips:Socket_Strip_Straight_1x05_Pitch2.54mm
Changed lines of the file:
@@
 F 0 "DD2" H 9100 3950 60  0000 C CNN
 F 1 "LIS331" H 9750 3950 60  0000 C CNN
-F 2 "LQFP_TQFP:LQFP48" H 9450 3450 60  0001 C CNN
+F 2 "LGA:16_3X3" H 9450 3450 60  0001 C CNN
 F 3 "" H 9450 3450 60  0000 C CNN
 	1    9450 3450
@@
 F 0 "XL3" V 1300 5950 40  0000 C CNN
 F 1 "CONN_2" V 1400 5950 40  0000 C CNN
-F 2 "Connectors:PLS-2" H 1350 5950 60  0001 C CNN
+F 2 "Installation:BH-6_CR2032" H 1350 5950 60  0001 C CNN
 F 3 "" H 1350 5950 60  0000 C CNN
 	1    1350 5950
@@
 F 0 "SW1" H 2000 6100 60  0000 C CNN
 F 1 "SWITCH" H 2350 6100 60  0000 C CNN
-F 2 "" H 2250 5850 60  0001 C CNN
+F 2 "Socket_Strips:Socket_Strip_Straight_1x03_Pitch2.54mm" H 2250 5850 60  0001 C CNN
 F 3 "" H 2250 5850 60  0000 C CNN
 	1    2250 5850
@@
 F 0 "C1" H 2650 6000 50  0000 L CNN
 F 1 "0.1u" H 2650 6200 50  0000 L CNN
-F 2 "Capacitors:CAP_0603" V 2850 5950 28  0000 C BNN
+F 2 "Capacitors:CAP_0805" V 2850 5950 28  0000 C BNN
 F 3 "" H 2750 6100 60  0000 C CNN
 	1    2750 6100
@@
 F 0 "L1" V 3250 5710 40  0000 C CNN
 F 1 "L" V 3250 5850 40  0000 C CNN
-F 2 "" V 3410 5860 40  0001 C CNN
+F 2 "Inductors:CD_type_6.0X5.5" V 3410 5860 40  0001 C CNN
 F 3 "" H 3350 5850 60  0000 C CNN
 	1    3350 5850
@@
 F 0 "XL2" H 1150 1750 60  0000 C CNN
 F 1 "ST_SWD" H 1500 1750 60  0000 C CNN
-F 2 "Connectors:PLS-4" H 1300 1450 60  0001 C CNN
+F 2 "Socket_Strips:Socket_Strip_Straight_1x04_Pitch2.54mm" H 1300 1450 60  0001 C CNN
 F 3 "" H 1300 1450 60  0000 C CNN
 	1    1300 1450
@@
 F 0 "XL4" V 10600 1500 50  0000 C CNN
 F 1 "CONN_5" V 10700 1500 50  0000 C CNN
-F 2 "Connectors:PLS-5" H 10650 1500 60  0001 C CNN
+F 2 "Socket_Strips:Socket_Strip_Straight_1x05_Pitch2.54mm" H 10650 1500 60  0001 C CNN
 F 3 "" H 10650 1500 60  0000 C CNN
 	1    10650 1500
@@
 F 0 "XL1" V 1150 2400 40  0000 C CNN
 F 1 "CONN_2" V 1250 2400 40  0000 C CNN
-F 2 "Connectors:PLS-2" H 1200 2400 60  0001 C CNN
+F 2 "Socket_Strips:Socket_Strip_Straight_1x02_Pitch2.54mm" H 1200 2400 60  0001 C CNN
 F 3 "" H 1200 2400 60  0000 C CNN
 	1    1200 2400

Commit message: Proceed PCB
Parts:
- C1: footprint Capacitors:CAP_0805 -> Capacitors:CAP_0603
Changed lines of the file:
@@
 F 0 "C1" H 2650 6000 50  0000 L CNN
 F 1 "0.1u" H 2650 6200 50  0000 L CNN
-F 2 "Capacitors:CAP_0805" V 2850 5950 28  0000 C BNN
+F 2 "Capacitors:CAP_0603" V 2850 5950 28  0000 C BNN
 F 3 "" H 2750 6100 60  0000 C CNN
 	1    2750 6100

Commit message: Increase PCB size
Parts:
- added HOLE? (x2): HOLE_METALLED, symbol HOLE_METALLED
Connections:
- net GND: now also HOLE?.H, HOLE?.H
Changed lines of the file:
@@
 	0    1    1    0
 $EndComp
+$Comp
+L HOLE_METALLED HOLE?
+U 1 1 592C6B25
+P 9800 5700
+F 0 "HOLE?" H 9300 5650 60  0000 C CNN
+F 1 "HOLE_METALLED" H 9250 5750 60  0000 C CNN
+F 2 "" H 9800 5700 60  0000 C CNN
+F 3 "" H 9800 5700 60  0000 C CNN
+	1    9800 5700
+	0    1    1    0
+$EndComp
+$Comp
+L HOLE_METALLED HOLE?
+U 1 1 592C6D1A
+P 10050 5700
+F 0 "HOLE?" H 9550 5650 60  0000 C CNN
+F 1 "HOLE_METALLED" H 9500 5750 60  0000 C CNN
+F 2 "" H 10050 5700 60  0000 C CNN
+F 3 "" H 10050 5700 60  0000 C CNN
+	1    10050 5700
+	0    1    1    0
+$EndComp
+$Comp
+L GND #PWR?
+U 1 1 592C6EB9
+P 9800 6150
+F 0 "#PWR?" H 9890 6130 30  0001 C CNN
+F 1 "GND" H 9800 6070 30  0001 C CNN
+F 2 "" H 9800 6150 60  0000 C CNN
+F 3 "" H 9800 6150 60  0000 C CNN
+	1    9800 6150
+	1    0    0    -1
+$EndComp
+$Comp
+L GND #PWR?
+U 1 1 592C6F17
+P 10050 6150
+F 0 "#PWR?" H 10140 6130 30  0001 C CNN
+F 1 "GND" H 10050 6070 30  0001 C CNN
+F 2 "" H 10050 6150 60  0000 C CNN
+F 3 "" H 10050 6150 60  0000 C CNN
+	1    10050 6150
+	1    0    0    -1
+$EndComp
+Wire Wire Line
+	10050 6150 10050 6000
+Wire Wire Line
+	9800 6150 9800 6000
 $EndSCHEMATC

Commit message: PCB start
Parts:
- HOLE1, HOLE2: renamed from HOLE?; footprint (none) -> PCB:Hole3_5_out6mm
Changed lines of the file:
@@
 $EndComp
 $Comp
-L HOLE_METALLED HOLE?
+L HOLE_METALLED HOLE1
 U 1 1 592C6B25
 P 9800 5700
-F 0 "HOLE?" H 9300 5650 60  0000 C CNN
+F 0 "HOLE1" H 9300 5650 60  0000 C CNN
 F 1 "HOLE_METALLED" H 9250 5750 60  0000 C CNN
-F 2 "" H 9800 5700 60  0000 C CNN
+F 2 "PCB:Hole3_5_out6mm" H 9800 5700 60  0001 C CNN
 F 3 "" H 9800 5700 60  0000 C CNN
 	1    9800 5700
@@
 $EndComp
 $Comp
-L HOLE_METALLED HOLE?
+L HOLE_METALLED HOLE2
 U 1 1 592C6D1A
 P 10050 5700
-F 0 "HOLE?" H 9550 5650 60  0000 C CNN
+F 0 "HOLE2" H 9550 5650 60  0000 C CNN
 F 1 "HOLE_METALLED" H 9500 5750 60  0000 C CNN
-F 2 "" H 10050 5700 60  0000 C CNN
+F 2 "PCB:Hole3_5_out6mm" H 10050 5700 60  0001 C CNN
 F 3 "" H 10050 5700 60  0000 C CNN
 	1    10050 5700
@@
 $EndComp
 $Comp
-L GND #PWR?
+L GND #PWR029
 U 1 1 592C6EB9
 P 9800 6150
-F 0 "#PWR?" H 9890 6130 30  0001 C CNN
+F 0 "#PWR029" H 9890 6130 30  0001 C CNN
 F 1 "GND" H 9800 6070 30  0001 C CNN
 F 2 "" H 9800 6150 60  0000 C CNN
@@
 $EndComp
 $Comp
-L GND #PWR?
+L GND #PWR030
 U 1 1 592C6F17
 P 10050 6150
-F 0 "#PWR?" H 10140 6130 30  0001 C CNN
+F 0 "#PWR030" H 10140 6130 30  0001 C CNN
 F 1 "GND" H 10050 6070 30  0001 C CNN
 F 2 "" H 10050 6150 60  0000 C CNN
